Commit message: fixed everything for the lidar and dimensions

File: urdf/hammerhead.urdf (robot description, URDF)
Before this commit: robot hammerhead, 2 links, 1 joints
Links:
- added link lidar; visual cylinder length=0.0105 radius=0.0325
- added link lidar_base; visual cylinder length=0.039 radius=0.0325
- added link rear_platform; visual box size=0.129 0.080 0.070
Joints:
- added joint lidar_base_joint: type fixed, parent rear_platform, child lidar_base, origin xyz=0.030 0 0.0545
- added joint lidar_joint: type continuous, parent lidar_base, child lidar, origin xyz=0 0 .0195, axis 0 0 1
- added joint rear_plat_joint: type fixed, parent base_link, child rear_platform, origin xyz=0.069 0 0.035
